File: Electronics/LED Array/LED Array.kicad_pcb (KiCad board)
At the start: 2 copper layers, 150 x 184.5 mm, 204 parts, among them J1 B2B-XH-A(LF)(SN), J2 B2B-XH-A(LF)(SN), J3 B2B-XH-A(LF)(SN), J4 B2B-XH-A(LF)(SN)

Commit message: led array IR-LED update:
Parts:
- removed J2, J3: B2B-XH-A(LF)(SN), AdditionalPartLibraries:JST_B2B-XH-A(LF)(SN)
- removed J4: B2B-XH-A(LF)(SN), Additional-parts:JST_B2B-XH-A(LF)(SN)
- added G***: LOGO, Additional-parts:Logo(Small), F.Cu at (208.2, 52.5)
- J1: value B2B-XH-A(LF)(SN) -> 282841-5; footprint AdditionalPartLibraries:JST_B2B-XH-A(LF)(SN) -> Additional-parts:TE_282841-5
- moved J1 5.14 mm to (159.4, 96.7), turned to 90 degrees
Connections:
- D1 pad 1: (no net) -> Net-(D1-Pad1) (x19)
- D5 pad 1: (no net) -> Net-(D5-Pad1) (x19)
- D5 pad 2: (no net) -> Net-(D1-Pad1) (x19)
- D6 pad 1: (no net) -> Net-(D6-Pad1) (x19)
- D6 pad 2: (no net) -> Net-(D5-Pad1) (x19)
- J1 pad 2: GND -> /Green12VPWM
- R1 pad 1: (no net) -> GND (x19)
- R1 pad 2: (no net) -> Net-(D6-Pad1) (x19)
Routing:
- net (no net): track 932.3 -> 0.00 mm
- net Net-(D1-Pad1): track 20.8 -> 418.2 mm
- net Net-(D5-Pad1): track 20.3 -> 406.7 mm
- net Net-(D6-Pad1): track 7.91 -> 156.3 mm
- net /IR12VPWM: track 396.5 -> 411.1 mm, vias 1 -> 2
- net /Blue12VPWM: track 482.4 -> 489.4 mm
- net /Green12VPWM: track 538.0 -> 541.7 mm
- net /Red12VPWM: track 595.3 -> 597.0 mm
- net Net-(D2-Pad3): track 386.6 -> 385.1 mm
- net Net-(D2-Pad1): track 385.3 -> 386.4 mm
- net GND: vias 28 -> 26
Other:
- board text added: "GND"
- board text added: "IR"
