File: electronics/phenobottle/phenobottle.kicad_sch (KiCad schematic)
At the start: 23 parts, among them J5 Conn_01x05_Socket, J6 TBP02R2-381-04BE, U2 STM32L432KCU6, U5 ITS716G, Y1 ECS-.327-12.5-34R-C-TR

Commit message: Added compute module and LED driver
Need to change 5V regulator for higher current as compute module needs
around 1 A with no peripherials (perhaps AP63205WU-7).
Parts:
- removed J6: TBP02R2-381-04BE, connectors:TBP02R2-381-04BE, symbol connectors:TBP02R2-381-04BE
- removed U5: ITS716G, Package_SO:SOIC-20W_7.5x12.8mm_P1.27mm, symbol Driver_FET:ITS716G
Connections:
- no-connect marks 4 -> 2
Other:
- added sheet COMPUTE (COMPUTE.kicad_sch)
- added sheet LED_DRIVER (led_driver.kicad_sch)
- note removed: "2 A each Channel"
- note removed: "Digital Output"
- moved on the sheet: J5
